Commit message: Add curriculum management and grasp offset calibration scripts

File: source/eggtart_grasp/eggtart_grasp/assets/urdf/robot.urdf (robot description, URDF)
Before this commit: robot generated_robot, 11 links, 10 joints
Links:
- link base_link: mass 1.23694208 -> 8.0
- link wheel_001: mass 1 -> 0.0819442; geometry collision mesh filename=meshes/part_045_solid_045.stl scale=0.001 0.001 0.001; visual mesh filename=meshes/part_045_solid_045.stl scale=0.001 0.001 0.001
- link wheel_002: mass 0.16388837 -> 0.08194418; geometry collision mesh filename=meshes/part_042_solid_042.stl scale=0.001 0.001 0.001; visual mesh filename=meshes/part_042_solid_042.stl scale=0.001 0.001 0.001
Joints:
- joint end_effector_joint: limit lower=-1.57 upper=1.57 effort=10 velocity=5 -> lower=-0.2 upper=1.57 effort=10 velocity=5
- joint link_002_joint: limit lower=-3.14 upper=1.57 effort=10 velocity=5 -> lower=-3.92 upper=0.0 effort=10 velocity=5
- joint link_003_joint: limit lower=-1.57 upper=1.57 effort=10 velocity=5 -> lower=0.0 upper=3.14 effort=10 velocity=5
- joint link_004_joint: limit lower=-1.57 upper=1.57 effort=10 velocity=5 -> lower=-3.14 upper=0.0 effort=10 velocity=5
